File: kicad/PowerSupply.sch (KiCad schematic (older format))
At the start: 25 parts, among them IC1 TPSM53604RDAR, IC2 LD39100PU33R, J1 Screw_Terminal_01x02, J2 Conn_01x01, J3 Conn_01x01, J4 Conn_01x02, J5 Conn_01x01, J6 Conn_01x02

Commit message: Power supply layout
Parts:
- removed J1: Screw_Terminal_01x02, TerminalBlock:TerminalBlock_Altech_AK300-2_P5.00mm, symbol Connector:Screw_Terminal_01x02
- removed L1: NLCV32T-R33M-EFR, IND_NLCV32TR_TDK, symbol 2021-01-12_17-35-09:NLCV32T-R33M-EFR
- added C4: C3216X5R1H106K160AB, SamacSys_Parts:CAPC3216X180N, symbol SamacSys_Parts:C3216X5R1H106K160AB
- added C6: GRM32EC81C476KE15L, SamacSys_Parts:CAPC3225X270N, symbol SamacSys_Parts:GRM32EC81C476KE15L
- added J1: 1935161, SamacSys_Parts:1701023, symbol SamacSys_Parts:1935161
- added J2: Conn_01x01, Connector_PinHeader_2.54mm:PinHeader_1x01_P2.54mm_Vertical, symbol Connector_Generic:Conn_01x01
- added L1: DFE201612P-R33M=P2, SamacSys_Parts:1286ASH1R0MP2, symbol SamacSys_Parts:DFE201612P-R33M=P2
- renumbered C8 to C10, C4 to C5, C5 to C7, C6 to C8, C7 to C9, J2 to J3, J3 to J4, J4 to J5, J5 to J6, J6 to J7
Connections:
- wire segments 96 -> 104
